Commit message: change suction to gripper

File: ravens/assets/ur5/ur5-gripper.urdf (robot description, URDF)
Before this commit: robot ur5, 13 links, 12 joints
Links:
- link ee_link: geometry collision box size=0.01 0.01 0.01
Joints:
- joint ee_fixed_joint: origin xyz=0.0 0.0823 0.0 rpy=-1.5707963267948966 0.0 0.0 -> xyz=0.0 0.0823 0.0 rpy=0.0 0.0 1.57079632679
- joint tool0-tool_tip: origin xyz=0 0 0.15 rpy=0 0 0 -> xyz=0 0 0 rpy=0 0 0

Commit message: final version

File: ravens/assets/ur5/ur5-gripper.urdf (robot description, URDF)
Before this commit: robot ur5, 13 links, 12 joints
Links:
- link base_link: geometry collision mesh filename=collision/base.stl; visual mesh filename=visual/base.stl
- link forearm_link: geometry collision mesh filename=collision/forearm.stl; visual mesh filename=visual/forearm.stl
- link shoulder_link: geometry collision mesh filename=collision/shoulder.stl; visual mesh filename=visual/shoulder.stl
- link upper_arm_link: geometry collision mesh filename=collision/upperarm.stl; visual mesh filename=visual/upperarm.stl
- link wrist_1_link: geometry collision mesh filename=collision/wrist1.stl; visual mesh filename=visual/wrist1.stl
- link wrist_2_link: geometry collision mesh filename=collision/wrist2.stl; visual mesh filename=visual/wrist2.stl
